Commit message: reconfigure

File: cartographer_ros/urdf/backpack_3d.urdf (robot description, URDF)
Before this commit: robot cartographer_backpack_3d, 4 links, 3 joints
Joints:
- joint horizontal_vlp16_link_joint: origin xyz=0.01 0. 0.19 rpy=0. -0.1745 3.1416 -> xyz=0.04 -0.17 0.06 rpy=0. -0.0 0.
- joint vertical_vlp16_link_joint: origin xyz=0.19 0. 0.04 rpy=0. 1.3963 0. -> xyz=0.15 -0.17 -0.1 rpy=1.309 0. 1.57
